File: HAM-Key.kicad_sch (KiCad schematic)
At the start: 33 parts, among them J1 USB_C_Receptacle_PowerOnly_6P, J2 Conn_01x04, Q1 DTC143Z, SW1 SW_Push, SW2 SW_SPDT, SW3 SW_SPDT, SW4 SW_SPDT, U3 ME4064AM5G, U4 ME6206A33XG

Commit message: temp commit
Parts:
- BZ1: footprint (none) -> Buzzer_Beeper:Buzzer_12x9.5RM7.6
- D1, D2, D3: footprint (none) -> LED_SMD:LED_0402_1005Metric_Pad0.77x0.64mm_HandSolder
- Q1: footprint (none) -> Package_TO_SOT_SMD:SOT-23-3
- SW2, SW3, SW4: footprint (none) -> nigh_Library:SS12D06G5
- U2: footprint (none) -> nigh_Library:nRF52810_module
Changed lines of the file:
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@@
   (junction (at 96.52 162.56) (diameter 0) (color 0 0 0 0)
   )
+  (junction (at 69.85 162.56) (diameter 0) (color 0 0 0 0)
+  )
   (junction (at 53.34 72.39) (diameter 0) (color 0 0 0 0)
   )
@@
   (junction (at 57.15 82.55) (diameter 0) (color 0 0 0 0)
   )
-  (junction (at 69.85 163.83) (diameter 0) (color 0 0 0 0)
-  )
   (junction (at 105.41 59.69) (diameter 0) (color 0 0 0 0)
   )
@@
     (stroke (width 0) (type default))
   )
-  (wire (pts (xy 62.23 163.83) (xy 69.85 163.83))
+  (wire (pts (xy 62.23 162.56) (xy 69.85 162.56))
     (stroke (width 0) (type default))
   )
@@
     (stroke (width 0) (type default))
   )
-  (wire (pts (xy 69.85 160.02) (xy 69.85 163.83))
+  (wire (pts (xy 69.85 160.02) (xy 69.85 162.56))
     (stroke (width 0) (type default))
   )
@@
     (stroke (width 0) (type default))
   )
-  (wire (pts (xy 62.23 160.02) (xy 62.23 163.83))
+  (wire (pts (xy 62.23 160.02) (xy 62.23 162.56))
     (stroke (width 0) (type default))
   )
@@
     (stroke (width 0) (type default))
   )
-  (wire (pts (xy 69.85 163.83) (xy 69.85 166.37))
-    (stroke (width 0) (type default))
-  )
   (wire (pts (xy 88.9 87.63) (xy 88.9 96.52))
     (stroke (width 0) (type default))
@@
   )
   (wire (pts (xy 85.09 134.62) (xy 99.06 134.62))
+    (stroke (width 0) (type default))
+  )
+  (wire (pts (xy 69.85 162.56) (xy 69.85 166.37))
     (stroke (width 0) (type default))
   )
@@
       (effects (font (size 1.27 1.27)))
     )
-    (property "Footprint" "" (at 137.16 120.65 0)
+    (property "Footprint" "LED_SMD:LED_0402_1005Metric_Pad0.77x0.64mm_HandSolder" (at 137.16 120.65 0)
       (effects (font (size 1.27 1.27)) hide)
     )
@@
       (effects (font (size 1.27 1.27)))
     )
-    (property "Footprint" "" (at 137.16 130.81 0)
+    (property "Footprint" "LED_SMD:LED_0402_1005Metric_Pad0.77x0.64mm_HandSolder" (at 137.16 130.81 0)
       (effects (font (size 1.27 1.27)) hide)
     )
@@
       (effects (font (size 1.27 1.27)))
     )
-    (property "Footprint" "" (at 194.31 49.53 0)
+    (property "Footprint" "nigh_Library:SS12D06G5" (at 194.31 49.53 0)
       (effects (font (size 1.27 1.27)) hide)
     )
@@
       (effects (font (size 1.27 1.27)))
     )
-    (property "Footprint" "" (at 68.58 40.64 0)
+    (property "Footprint" "nigh_Library:nRF52810_module" (at 68.58 40.64 0)
       (effects (font (size 1.27 1.27)) hide)
     )
@@
       (effects (font (size 1.27 1.27)))
     )
-    (property "Footprint" "" (at 210.82 120.65 0)
+    (property "Footprint" "nigh_Library:SS12D06G5" (at 210.82 120.65 0)
       (effects (font (size 1.27 1.27)) hide)
     )
@@
       (effects (font (size 1.27 1.27)) (justify right))
     )
-    (property "Footprint" "" (at 215.9 141.605 90)
+    (property "Footprint" "Buzzer_Beeper:Buzzer_12x9.5RM7.6" (at 215.9 141.605 90)
       (effects (font (size 1.27 1.27)) hide)
     )
@@
       (effects (font (size 1.27 1.27)) (justify left))
     )
-    (property "Footprint" "" (at 149.86 97.79 0)
+    (property "Footprint" "Package_TO_SOT_SMD:SOT-23-3" (at 149.86 97.79 0)
       (effects (font (size 1.27 1.27)) (justify left) hide)
     )
@@
       (effects (font (size 1.27 1.27)))
     )
-    (property "Footprint" "" (at 137.16 125.73 0)
+    (property "Footprint" "LED_SMD:LED_0402_1005Metric_Pad0.77x0.64mm_HandSolder" (at 137.16 125.73 0)
       (effects (font (size 1.27 1.27)) hide)
     )
@@
       (effects (font (size 1.27 1.27)))
     )
-    (property "Footprint" "" (at 210.82 130.81 0)
-      (effects (font (size 1.27 1.27)) hide)
-    )
+    (property "Footprint" "nigh_Library:SS12D06G5" (at 210.82 130.81 0)
+      (effects (font (size 1.27 1.27)) hide)
+    )

Commit message: update
Parts:
- removed R9: 800k, Resistor_SMD:R_0402_1005Metric_Pad0.72x0.64mm_HandSolder, symbol Device:R_Small
- removed U3: ME4064AM5G, symbol nigh_Library:ME4064AM5G
- removed U4: ME6206A33XG, symbol nigh_Library:ME6206A33XG
- added C5, C6: 1uF, Capacitor_SMD:C_0603_1608Metric_Pad1.08x0.95mm_HandSolder, symbol Device:C_Small
- added D4: BLUE, LED_SMD:LED_0402_1005Metric_Pad0.77x0.64mm_HandSolder, symbol Device:LED
- added D5: RED, LED_SMD:LED_0402_1005Metric_Pad0.77x0.64mm_HandSolder, symbol Device:LED
- added H1, H2, H3, H4: M3.5, MountingHole:MountingHole_3.5mm_Pad_Via, symbol Mechanical:MountingHole
- added R12, R13: 1k, Resistor_SMD:R_0402_1005Metric_Pad0.72x0.64mm_HandSolder, symbol Device:R_Small
- added U2: ~, Package_DFN_QFN:DFN-8-1EP_3x3mm_P0.65mm_EP1.55x2.4mm, symbol nigh_Library:LP4073
- added U3: ~, Package_TO_SOT_SMD:TSOT-23_HandSoldering, symbol nigh_Library:WL9100S3
- BATT1: renamed from BT1; footprint (none) -> nigh_Library:BATT2030
- BZ1: footprint Buzzer_Beeper:Buzzer_12x9.5RM7.6 -> nigh_Library:buzzer_SMD
- D1: value LED -> RED
- D2: value LED -> BLUE
- D3: value LED -> WHITE
- R14: value 330R -> 0R
- R15: renamed from R3; value X -> 10k
- SW3: renamed from SW2; footprint nigh_Library:SS12D06G5 -> nigh_Library:MSK12
- SW4: renamed from SW3; footprint nigh_Library:SS12D06G5 -> nigh_Library:MSK12
- USB1: renamed from J1; footprint (none) -> nigh_Library:Type-C-3.2H
- renumbered C2 to C1, C3 to C2, C1 to C3, R7 to R1, R12 to R10, R13 to R11, R8 to R2, R1 to R3, R2 to R4, R4 to R5, R5 to R6, R6 to R7, R10 to R8, R11 to R9, SW4 to SW2, U2 to U1
Connections:
- net +3.3V: now also U3.3 (VOUT)
- net +5V: now also C6.1, D4.2 (A), D5.2 (A), U2.8 (IN)
- net BAT+: now also C5.1, U3.2 (VIN)
- net CC1: now also R6.2; no longer R5.2
- net CC2: now also R5.2; no longer R6.2
- net GND: now also C5.2, C6.2, U2.4 (EN), U2.5 (GND), U3.1 (GND)
- net at BATT1.1 (+), SW2.2 (B), SW2.3 (C): now also U2.1 (BAT)
- net at R15.1: now also U2.6 (ISET)
- new net: D5.1 (K), R13.1
- new net: D4.1 (K), R12.1
- new net: R12.2, U2.2 (FULL)
- new net: R13.2, U2.3 (CHRG)
Other:
- moved on the sheet: J2, R15

Commit message: fix some issue
Parts:
- added C7: 1uF, Capacitor_SMD:C_0603_1608Metric_Pad1.08x0.95mm_HandSolder, symbol Device:C_Small
- added C8: 4.7uF, Capacitor_SMD:C_0603_1608Metric_Pad1.08x0.95mm_HandSolder, symbol Device:C_Small
- R10, R11, R9: value 330R -> 470R
- R14: value 0R -> 100R
- R5: value 10R -> NC; now left out of the parts list
Connections:
- net +3.3V: now also U3.2 (VOUT), C8.1; no longer U3.3 (VOUT)
- net BAT+: now also U3.3 (VIN); no longer U3.2 (VIN)
- net GND: now also C7.1, C8.2
- net at BATT1.1 (+), SW2.2 (B), SW2.3 (C)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: now also C7.2
Changed lines of the file:
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@@
 (kicad_sch (version 20230121) (generator eeschema)
   (paper "A4")
+  (junction (at 232.41 46.99) (diameter 0) (color 0 0 0 0)
+  )
   (junction (at 241.3 73.66) (diameter 0) (color 0 0 0 0)
   )
@@
   (junction (at 130.81 144.78) (diameter 0) (color 0 0 0 0)
   )
+  (junction (at 232.41 86.36) (diameter 0) (color 0 0 0 0)
+  )
   (junction (at 57.15 72.39) (diameter 0) (color 0 0 0 0)
   )
   (junction (at 189.23 59.69) (diameter 0) (color 0 0 0 0)
   )
+  (junction (at 209.55 73.66) (diameter 0) (color 0 0 0 0)
+  )
   (junction (at 57.15 82.55) (diameter 0) (color 0 0 0 0)
   )
@@
     (stroke (width 0) (type default))
   )
+  (wire (pts (xy 232.41 46.99) (xy 241.3 46.99))
+    (stroke (width 0) (type default))
+  )
   (wire (pts (xy 57.15 81.28) (xy 57.15 82.55))
     (stroke (width 0) (type default))
@@
     (stroke (width 0) (type default))
   )
+  (wire (pts (xy 232.41 86.36) (xy 232.41 88.9))
+    (stroke (width 0) (type default))
+  )
   (wire (pts (xy 207.01 76.2) (xy 210.82 76.2))
     (stroke (width 0) (type default))
@@
     (stroke (width 0) (type default))
   )
+  (wire (pts (xy 209.55 73.66) (xy 210.82 73.66))
+    (stroke (width 0) (type default))
+  )
   (wire (pts (xy 83.82 87.63) (xy 83.82 99.06))
     (stroke (width 0) (type default))
@@
     (stroke (width 0) (type default))
   )
+  (wire (pts (xy 232.41 46.99) (xy 232.41 48.26))
+    (stroke (width 0) (type default))
+  )
   (wire (pts (xy 53.34 72.39) (xy 57.15 72.39))
     (stroke (width 0) (type default))
   )
+  (wire (pts (xy 218.44 54.61) (xy 232.41 54.61))
+    (stroke (width 0) (type default))
+  )
   (wire (pts (xy 212.09 147.32) (xy 215.9 147.32))
     (stroke (width 0) (type default))
@@
     (stroke (width 0) (type default))
   )
+  (wire (pts (xy 209.55 73.66) (xy 209.55 86.36))
+    (stroke (width 0) (type default))
+  )
   (wire (pts (xy 218.44 53.34) (xy 218.44 54.61))
     (stroke (width 0) (type default))
@@
     (stroke (width 0) (type default))
   )
-  (wire (pts (xy 232.41 81.28) (xy 232.41 88.9))
+  (wire (pts (xy 232.41 81.28) (xy 232.41 86.36))
     (stroke (width 0) (type default))
   )
@@
     (stroke (width 0) (type default))
   )
+  (wire (pts (xy 209.55 86.36) (xy 217.17 86.36))
+    (stroke (width 0) (type default))
+  )
   (wire (pts (xy 180.34 59.69) (xy 189.23 59.69))
     (stroke (width 0) (type default))
@@
     (stroke (width 0) (type default))
   )
+  (wire (pts (xy 222.25 86.36) (xy 232.41 86.36))
+    (stroke (width 0) (type default))
+  )
   (wire (pts (xy 215.9 133.35) (xy 220.98 133.35))
     (stroke (width 0) (type default))
@@
     (stroke (width 0) (type default))
   )
-  (wire (pts (xy 228.6 46.99) (xy 241.3 46.99))
+  (wire (pts (xy 228.6 46.99) (xy 232.41 46.99))
     (stroke (width 0) (type default))
   )
@@
     (stroke (width 0) (type default))
   )
-  (wire (pts (xy 189.23 73.66) (xy 210.82 73.66))
+  (wire (pts (xy 232.41 54.61) (xy 232.41 53.34))
     (stroke (width 0) (type default))
   )
@@
   )
   (wire (pts (xy 215.9 123.19) (xy 220.98 123.19))
+    (stroke (width 0) (type default))
+  )
+  (wire (pts (xy 189.23 73.66) (xy 209.55 73.66))
     (stroke (width 0) (type default))
   )
@@
   )
   (symbol (lib_id "Device:R_Small") (at 110.49 54.61 90) (unit 1)
-    (in_bom yes) (on_board yes) (dnp no)
+    (in_bom no) (on_board yes) (dnp no)
     (property "Reference" "R5" (at 111.76 54.61 90)
       (effects (font (size 1.27 1.27)) (justify left))
     )
-    (property "Value" "10R" (at 115.57 55.88 90)
+    (property "Value" "NC" (at 115.57 55.88 90)
       (effects (font (size 1.27 1.27)) (justify left))
     )
@@
   (symbol (lib_id "Device:LED") (at 194.31 78.74 180) (unit 1)
     (in_bom yes) (on_board yes) (dnp no)
-    (property "Reference" "D5" (at 196.85 80.01 0)
-      (effects (font (size 1.27 1.27)))
-    )
-    (property "Value" "RED" (at 190.5 77.47 0)
+    (property "Reference" "D5" (at 191.77 77.47 0)
+      (effects (font (size 1.27 1.27)))
+    )
+    (property "Value" "RED" (at 186.69 77.47 0)
       (effects (font (size 1.27 1.27)))
     )
@@
       (effects (font (size 1.27 1.27)) (justify left))
     )
-    (property "Value" "0R" (at 214.63 148.59 90)
+    (property "Value" "100R" (at 215.9 148.59 90)
       (effects (font (size 1.27 1.27)) (justify left))
     )
@@
       (effects (font (size 1.27 1.27)) (justify left))
     )
-    (property "Value" "330R" (at 153.67 121.92 90)
+    (property "Value" "470R" (at 153.67 121.92 90)
       (effects (font (size 1.27 1.27)) (justify left))
     )
@@
   (symbol (lib_id "Device:LED") (at 194.31 76.2 180) (unit 1)
     (in_bom yes) (on_board yes) (dnp no)
-    (property "Reference" "D4" (at 196.85 77.47 0)
-      (effects (font (size 1.27 1.27)))
-    )
-    (property "Value" "BLUE" (at 190.5 74.93 0)
+    (property "Reference" "D4" (at 191.77 74.93 0)
+      (effects (font (size 1.27 1.27)))
+    )
+    (property "Value" "BLUE" (at 186.69 74.93 0)
       (effects (font (size 1.27 1.27)))
     )
@@
       (effects (font (size 1.27 1.27)) (justify left))
     )
-    (property "Value" "330R" (at 153.67 127 90)
+    (property "Value" "470R" (at 153.67 127 90)
       (effects (font (size 1.27 1.27)) (justify left))
     )
@@
         (path "/613fe7f2-55f8-4770-afca-1b2f2a94adcb"
           (reference "H4") (unit 1)
+        )
+      )
+    )
+  )
+  (symbol (lib_id "Device:C_Small") (at 232.41 50.8 0) (unit 1)
+    (in_bom yes) (on_board yes) (dnp no)
+    (property "Reference" "C8" (at 233.68 49.53 90)
+      (effects (font (size 1.27 1.27)) (justify left))
+    )
+    (property "Value" "4.7uF" (at 231.14 55.88 90)
+      (effects (font (size 1.27 1.27)) (justify left))
+    )
+    (property "Footprint" "Capacitor_SMD:C_0603_1608Metric_Pad1.08x0.95mm_HandSolder" (at 232.41 50.8 0)
+      (effects (font (size 1.27 1.27)) hide)
+    )
+    (property "Datasheet" "~" (at 232.41 50.8 0)
+      (effects (font (size 1.27 1.27)) hide)
+    )
+    (pin "1")
+    (pin "2")
+    (instances
+      (project "HAM-Key"
+        (path "/613fe7f2-55f8-4770-afca-1b2f2a94adcb"
+          (reference "C8") (unit 1)
         )
       )
@@
     )
   )
+  (symbol (lib_id "Device:C_Small") (at 219.71 86.36 270) (unit 1)
+    (in_bom yes) (on_board yes) (dnp no)
+    (property "Reference" "C7" (at 220.98 87.63 90)
+      (effects (font (size 1.27 1.27)) (justify left))
+    )
+    (property "Value" "1uF" (at 214.63 85.09 90)
+      (effects (font (size 1.27 1.27)) (justify left))
+    )
+    (property "Footprint" "Capacitor_SMD:C_0603_1608Metric_Pad1.08x0.95mm_HandSolder" (at 219.71 86.36 0)
+      (effects (font (size 1.27 1.27)) hide)
+    )
+    (property "Datasheet" "~" (at 219.71 86.36 0)
+      (effects (font (size 1.27 1.27)) hide)
+    )
+    (pin "1")
+    (pin "2")
+    (instances
+      (project "HAM-Key"
+        (path "/613fe7f2-55f8-4770-afca-1b2f2a94adcb"
+          (reference "C7") (unit 1)
+        )
+      )
+    )
+  )
   (symbol (lib_id "Device:R_Small") (at 147.32 130.81 90) (unit 1)
     (in_bom yes) (on_board yes) (dnp no)
@@
       (effects (font (size 1.27 1.27)) (justify left))
     )
-    (property "Value" "330R" (at 153.67 132.08 90)
-      (effects (font (size 1.27 1.27)) (justify left))
-    )
+    (property "Value" "470R" (at 153.67 132.08 90)
+      (effects (font (size 1.27 1.27)) (justify left))
+    )
